Commit message: test

File: iiwa_description/urdf/iiwa14.xacro (robot description, xacro)
@@ -299,4 +299,12 @@
     <link name="${robot_name}_link_ee">
     </link>
+    <!--Cai: add camera frame -->
+    <joint name="${robot_name}_joint_camera" type="fixed">
+      <parent link="${robot_name}_link_ee"/>
+      <child link="${robot_name}_link_camera"/>
+      <origin xyz="0 0 0" rpy="0 0 0"/>
+    </joint>
+    <link name="${robot_name}_link_camera">
+    </link>
     <!--Extensions -->
     <xacro:iiwa_gazebo robot_name="${robot_name}" />
